File: PCB/Knox's rp2040 devboard.kicad_pcb (KiCad board)
At the start: 2 copper layers, 21 x 51 mm, 34 parts, among them J1 USB_C_Receptacle_USB2.0_14P, J2 Conn_01x20, J3 Conn_01x20, J4 Conn_01x03, SW1 SW_Push, U1 RP2040, U2 MCP1700x-330xxTT, U4 W25Q16JVZPIQ TR, Y1 12 MHz

Commit message: a
Other:
- board text added: "Knox's RP2040 Dev Board"
Changed lines of the file:
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@@
 		(tags "Through hole pin header THT 1x03 2.54mm single row")
 		(property "Reference" "J4"
-			(at 2.385 2.665 180)
+			(at -0.065 -2.625 180)
 			(layer "F.SilkS")
 			(effects
@@
 		(layer "Edge.Cuts")
 	)
+	(gr_text "Knox's RP2040\nDev Board"
+		(at 185.22 103.78 0)
+		(layer "F.SilkS")
+		(effects
+			(font
+				(size 0.8 0.8)
+				(thickness 0.16)
+				(bold yes)
+			)
+			(justify left bottom)
+		)
+	)
 	(segment
